File: PCBs/integrated-serial-device/serial-hat.kicad_pcb (KiCad board)
At the start: 2 copper layers, 193 x 113 mm, 29 parts, among them CN1 Modem port, CN2 Modem out 3, CN3 Printer port, J1 Rpi headers, J3 Conn_01x02_Pin, K1 Quicktake, K2 ImageWriter, SW1 Modem To Proxy, SW2 Modem to Quicktake, SW3 Modem out 3, SW5 Printer to Proxy, SW6 Printer to ImageWriter, SW7 SW_SPST, SW8 SW_Slide_DPDT SHOU HAN MSK-22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, U1 MAX3232, U2 PC817C-S

Commit message: Update to new lib
Parts:
- added Unpopulated: 4PDT 12 pins Piano Switch, Colins-Kicad:4PDT 12 pins Piano Switch, F.Cu at (194.8, 78.8)
- CN1, CN2, CN3: footprint DIN5:CONN-TH_DIN-504-M10 -> Colins-Kicad:DIN-5-M C23689428
- K1, K2: footprint DIN5:MINI-DIN8 -> Colins-Kicad:MINI-DIN8-F C20611694
- SW1, SW2, SW3, SW5, SW6: footprint DIN5:4PDT piano switch -> Colins-Kicad:4PDT 12 pins Piano Switch
- SW7: footprint DIN5:SPST_power_switch -> Colins-Kicad:SPST momentary switch C6575016
- SW8: footprint DIN5:DPDT slide switch C7507433 -> Colins-Kicad:DPDT slide switch C7507433
- U2: footprint Package_SO:SOP-4_3.8x4.1mm_P2.54mm -> Colins-Kicad:PC817C-S C3008369
- moved U2 27.7 mm to (80.4, 111.9)
Routing:
- net FAN_CTRL: track 76.0 -> 127.8 mm, vias 1 -> 0
- net FAN_5V: track 45.9 -> 74.2 mm
- net 5V: track 49.6 -> 77.8 mm
- net PWR_LED: track 393.7 -> 391.8 mm
- net 3.3V: track 180.3 -> 179.3 mm
- net RX1_OUT_GPIO5: track 194.6 -> 194.0 mm
