File: PCBs/integrated-serial-device/serial-hat.kicad_sch (KiCad schematic)
At the start: 22 parts, among them CN1 Modem port, CN2 Modem out 3, CN3 Printer port, J1 Rpi headers, J3 Conn_01x02_Pin, K1 Quicktake, K2 ImageWriter, SW1 Modem To Proxy, SW2 Modem to Quicktake, SW3 Modem out 3, SW5 Printer to Proxy, SW6 Printer to ImageWriter, SW7 SW_SPST, SW8 SW_Slide_DPDT SHOU HAN MSK-22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, U1 MAX3232, U2 PC817C-S

Commit message: Update stls and notes
Connections:
- no-connect marks 47 -> 50
Changed lines of the file:
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@@
+	)
+	(no_connect
+		(at 99.06 24.13)
 	)
 	(no_connect
@@
 	)
 	(no_connect
+		(at 111.76 52.07)
+	)
+	(no_connect
 		(at 111.76 31.75)
 	)
 	(no_connect
+		(at 99.06 59.69)
+	)
+	(no_connect
