File: PCBs/qt-connector-mac/qt-connector.kicad_pcb (KiCad board)
At the start: 2 copper layers, 40.9 x 53 mm, 6 parts, among them K1 Quicktake, K2 Modem port, K3 Printer port, K4 ImageWriter

Commit message: Update to new lib
Parts:
- K1, K4: footprint DIN5:MINI-DIN8 -> Colins-Kicad:MINI-DIN8-F C20611694
- K2, K3: footprint DIN5:CONN-TH_DIN-504-M10 -> Colins-Kicad:DIN-5-M C23689428
