File: PCBs/serial-hat/serial-hat.kicad_sch (KiCad schematic)
At the start: 11 parts, among them CN1 Modem port, CN2 Printer port, J1 Conn_01x02_Pin, J7 Rpi headers, U1 PC817C-S, U2 MAX3232

Commit message: Update stls and notes
Parts:
- added SW7: SW_SPST, Colins-Kicad:SPST momentary switch C6575016, symbol Switch:SW_DIP_x01
Connections:
- net GND: now also SW7.2, SW7.3, SW7.4 (3)
- net PWR_BTN: now reaches J7.5 (Pin_5)
- net PWR_BTN: now also SW7.1
- no-connect marks 21 -> 24

Commit message: Add teardrops
Parts:
- CN1, CN2: LCSC C23689428 -> C2939346; Supplier Part C23689428 -> C2939346
Changed lines of the file:
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@@
 			)
 		)
-		(property "Supplier Part" "C23689428"
+		(property "Supplier Part" "C2939346"
 			(at 187.96 123.19 0)
 			(effects
@@
 			)
 		)
-		(property "LCSC" "C23689428"
+		(property "LCSC" "C2939346"
 			(at 187.96 123.19 0)
 			(effects
@@
 			)
 		)
-		(property "Supplier Part" "C23689428"
+		(property "Supplier Part" "C2939346"
 			(at 187.96 91.44 0)
 			(effects
@@
 			)
 		)
-		(property "LCSC" "C23689428"
-			(at 187.96 91.44 0)
-			(effects
+		(property "LCSC" "C2939346"
+			(at 187.96 91.44 0)
+			(effects
